File: quahog-2-routed.sch (EAGLE design)
At the start: 33 parts, among them IC3 MCP1703CB, IC5 24AA128SN, J1 AYZ0202, X1 16 MHz

Commit message: update
Connections:
- removed net VIN: BATTPOWER.S
- net PWR: now also BATTPOWER.S
Changed lines of the file:
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@@
 <label x="140.462" y="97.282" size="1.778" layer="95"/>
+</segment>
+<segment>
+<pinref part="BATTPOWER" gate="A" pin="S"/>
+<wire x1="425.196" y1="257.048" x2="432.308" y2="257.048" width="0.1524" layer="91"/>
+<wire x1="432.308" y1="257.048" x2="432.308" y2="259.588" width="0.1524" layer="91"/>
+<label x="432.054" y="260.858" size="1.778" layer="95"/>
 </segment>
 </net>
@@
 </segment>
 </net>
-<net name="VIN" class="0">
-<segment>
-<pinref part="BATTPOWER" gate="A" pin="S"/>
-<wire x1="425.196" y1="257.048" x2="432.308" y2="257.048" width="0.1524" layer="91"/>
-<wire x1="432.308" y1="257.048" x2="432.308" y2="259.588" width="0.1524" layer="91"/>
-<label x="432.054" y="260.858" size="1.778" layer="95"/>
-</segment>
-</net>

Commit message: update
Connections:
- removed net A4_SDA: ATMEGA328.PC4(ADC4/SDA), JP5.9
- removed net A5_SCL: ATMEGA328.PC5(ADC5/SCL), JP5.11
- net SCL: now also ATMEGA328.PC5(ADC5/SCL), JP5.11
- net SDA: now also ATMEGA328.PC4(ADC4/SDA), JP5.9
Changed lines of the file:
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@@
-</segment>
-</net>
-<net name="A4_SDA" class="0">
-<segment>
-<wire x1="80.01" y1="139.7" x2="91.44" y2="139.7" width="0.1524" layer="91"/>
-<label x="82.55" y="139.7" size="1.778" layer="95"/>
-<pinref part="ATMEGA328" gate="G$1" pin="PC4(ADC4/SDA)"/>
-</segment>
-<segment>
-<wire x1="-101.6" y1="238.76" x2="-106.68" y2="238.76" width="0.1524" layer="91"/>
-<label x="-114.3" y="238.76" size="1.778" layer="95"/>
-<pinref part="JP5" gate="A" pin="9"/>
 </segment>
 </net>
@@
 </segment>
 </net>
-<net name="A5_SCL" class="0">
-<segment>
-<wire x1="80.01" y1="137.16" x2="91.44" y2="137.16" width="0.1524" layer="91"/>
-<label x="82.55" y="137.16" size="1.778" layer="95"/>
-<pinref part="ATMEGA328" gate="G$1" pin="PC5(ADC5/SCL)"/>
-</segment>
-<segment>
-<wire x1="-101.6" y1="236.22" x2="-106.68" y2="236.22" width="0.1524" layer="91"/>
-<label x="-114.3" y="236.22" size="1.778" layer="95"/>
-<pinref part="JP5" gate="A" pin="11"/>
-</segment>
-</net>
 <net name="N$2" class="0">
 <segment>
@@
 <label x="248.412" y="238.252" size="1.778" layer="95"/>
 </segment>
+<segment>
+<wire x1="80.01" y1="139.7" x2="91.44" y2="139.7" width="0.1524" layer="91"/>
+<label x="82.55" y="139.7" size="1.778" layer="95"/>
+<pinref part="ATMEGA328" gate="G$1" pin="PC4(ADC4/SDA)"/>
+</segment>
+<segment>
+<wire x1="-101.6" y1="238.76" x2="-106.68" y2="238.76" width="0.1524" layer="91"/>
+<label x="-114.3" y="238.76" size="1.778" layer="95"/>
+<pinref part="JP5" gate="A" pin="9"/>
+</segment>
 </net>
 <net name="SCL" class="0">
@@
 <label x="214.122" y="245.872" size="1.778" layer="95"/>
 </segment>
-</net>
+<segment>
+<wire x1="80.01" y1="137.16" x2="91.44" y2="137.16" width="0.1524" layer="91"/>
+<label x="82.55" y="137.16" size="1.778" layer="95"/>
+<pinref part="ATMEGA328" gate="G$1" pin="PC5(ADC5/SCL)"/>
+</segment>
+<segment>
+<wire x1="-101.6" y1="236.22" x2="-106.68" y2="236.22" width="0.1524" layer="91"/>
+<label x="-114.3" y="236.22" size="1.778" layer="95"/>
+<pinref part="JP5" gate="A" pin="11"/>
+</segment>
+</net>
