File: quahog_0.1.0.brd (EAGLE design)
At the start: 71.3 x 17.9 mm, 33 parts, among them IC3 MCP1703CB, IC5 24AA128SN, J1 AYZ0202, X1 16 MHz

Commit message: update
Connections:
- removed net D10_SS: ATMEGA328.14
- net D10: now also ATMEGA328.14
Routing:
- net D10: track 0.00 -> 54.9 mm, vias 0 -> 4
- net D3: track 76.5 -> 89.4 mm, vias 3 -> 9
- net A3: track 24.2 -> 36.9 mm
- net A2: track 59.2 -> 46.6 mm, vias 5 -> 3
- net SDA: track 65.4 -> 52.9 mm
- net GND: track 193.5 -> 181.7 mm, vias 5 -> 7
- net N$1: track 3.66 -> 10.3 mm, vias 0 -> 2
- net D0_RX: track 22.6 -> 29.2 mm, vias 1 -> 3
- net N$4: track 34.9 -> 41.3 mm, vias 3 -> 4
- net AREF: track 62.8 -> 57.7 mm
- net VCC: track 109.9 -> 114.7 mm, vias 4 -> 10
- net A1: track 46.6 -> 42.2 mm, vias 2 -> 3
- net D4: track 16.6 -> 20.4 mm, vias 0 -> 2
- net RST: track 36.4 -> 32.7 mm, vias 1 -> 2
- net N$7: track 30.3 -> 32.9 mm, vias 1 -> 2
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Other:
- board size 71.3 x 17.9 mm -> 61.9 x 17.9 mm
