File: quahog_0.1.0.sch (EAGLE design)
At the start: 33 parts, among them IC3 MCP1703CB, IC5 24AA128SN, J1 AYZ0202, X1 16 MHz

Commit message: update
Connections:
- removed net D10_SS: ATMEGA328.PB2(SS/OC1B)
- net D10: now also ATMEGA328.PB2(SS/OC1B)
Changed lines of the file:
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@@
-</segment>
-</net>
-<net name="D10_SS" class="0">
-<segment>
-<wire x1="80.01" y1="99.06" x2="91.44" y2="99.06" width="0.1524" layer="91"/>
-<label x="82.55" y="99.06" size="1.778" layer="95"/>
-<pinref part="ATMEGA328" gate="G$1" pin="PB2(SS/OC1B)"/>
 </segment>
 </net>
@@
 <pinref part="JP5" gate="A" pin="6"/>
 <wire x1="-93.98" y1="243.84" x2="-88.9" y2="243.84" width="0.1524" layer="91"/>
-<label x="-88.9" y="243.84" size="1.778" layer="95"/>
-</segment>
-</net>
+<label x="-86.36" y="243.84" size="1.778" layer="95"/>
+</segment>
+<segment>
+<wire x1="80.01" y1="99.06" x2="91.44" y2="99.06" width="0.1524" layer="91"/>
+<label x="82.55" y="99.06" size="1.778" layer="95"/>
+<pinref part="ATMEGA328" gate="G$1" pin="PB2(SS/OC1B)"/>
+</segment>
+</net>
