File: quahog-0.1.0.sch (EAGLE design)
At the start: 33 parts, among them IC3 MCP1703CB, IC5 24AA128SN, J1 AYZ0202, X1 16 MHz

Commit message: update
Connections:
- removed net D10_SS: ATMEGA328.PB2(SS/OC1B)
- new net 3V3R: C3.1, C4.1, IC3.VO, J1.3, J2.7
- net D10: now also ATMEGA328.PB2(SS/OC1B)
- net VCC: no longer C3.1, C4.1, IC3.VO, J1.3, J2.7
Changed lines of the file:
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@@
 <part name="FRAME1" library="frames" deviceset="A4L-LOC" device="" value="Moteino"/>
 <part name="SUPPLY5" library="supply2" deviceset="GND" device=""/>
-<part name="SUPPLY3" library="SparkFun" deviceset="VCC" device="" value="3.3V"/>
 <part name="SUPPLY10" library="supply2" deviceset="GND" device=""/>
 <part name="SUPPLY14" library="supply2" deviceset="GND" device=""/>
@@
 <part name="SUPPLY8" library="supply2" deviceset="GND" device=""/>
 <part name="P+2" library="supply1" deviceset="VCC" device=""/>
-<part name="SUPPLY11" library="SparkFun" deviceset="VCC" device="" value="3.3V"/>
 <part name="J2" library="SparkFun-Connectors" deviceset="M07" device=""/>
-<part name="SUPPLY12" library="SparkFun" deviceset="VCC" device="" value="3.3V"/>
 <part name="P+4" library="supply1" deviceset="VCC" device=""/>
 <part name="J3" library="SparkFun-Connectors" deviceset="M02" device="PTH"/>
@@
 <instance part="FRAME1" gate="G$1" x="0" y="0"/>
 <instance part="SUPPLY5" gate="GND" x="19.05" y="124.46"/>
-<instance part="SUPPLY3" gate="1" x="193.04" y="76.2"/>
 <instance part="SUPPLY10" gate="GND" x="193.04" y="53.34"/>
 <instance part="SUPPLY14" gate="GND" x="29.21" y="88.9"/>
@@
 <instance part="SUPPLY8" gate="GND" x="289.56" y="83.82"/>
 <instance part="P+2" gate="VCC" x="340.36" y="91.44"/>
-<instance part="SUPPLY11" gate="1" x="289.56" y="91.44"/>
 <instance part="J2" gate="G$1" x="17.78" y="27.94"/>
-<instance part="SUPPLY12" gate="1" x="22.86" y="40.64"/>
 <instance part="P+4" gate="VCC" x="17.78" y="165.1"/>
 <instance part="J3" gate="G$1" x="358.14" y="25.4"/>
@@
 </segment>
 </net>
-<net name="D10_SS" class="0">
-<segment>
-<wire x1="80.01" y1="99.06" x2="91.44" y2="99.06" width="0.1524" layer="91"/>
-<label x="82.55" y="99.06" size="1.778" layer="95"/>
-<pinref part="ATMEGA328" gate="G$1" pin="PB2(SS/OC1B)"/>
-</segment>
-</net>
 <net name="RST" class="0">
 <segment>
@@
 <net name="VCC" class="0">
 <segment>
-<wire x1="193.04" y1="71.12" x2="200.66" y2="71.12" width="0.1524" layer="91"/>
-<wire x1="200.66" y1="71.12" x2="215.9" y2="71.12" width="0.1524" layer="91"/>
-<pinref part="IC3" gate="G$1" pin="VO"/>
-<pinref part="SUPPLY3" gate="1" pin="VCC"/>
-<wire x1="193.04" y1="71.12" x2="193.04" y2="76.2" width="0.2032" layer="91"/>
-<pinref part="C4" gate="G$1" pin="1"/>
-<junction x="193.04" y="71.12"/>
-<pinref part="C3" gate="G$1" pin="1"/>
-<junction x="200.66" y="71.12"/>
-</segment>
-<segment>
 <pinref part="IC5" gate="G$1" pin="VCC"/>
 <pinref part="P+3" gate="VCC" pin="VCC"/>
@@
 <wire x1="320.04" y1="88.9" x2="340.36" y2="88.9" width="0.1524" layer="91"/>
 <pinref part="P+2" gate="VCC" pin="VCC"/>
-</segment>
-<segment>
-<pinref part="J1" gate="G$1" pin="3"/>
-<wire x1="289.56" y1="91.44" x2="309.88" y2="91.44" width="0.1524" layer="91"/>
-<pinref part="SUPPLY11" gate="1" pin="VCC"/>
-</segment>
-<segment>
-<pinref part="J2" gate="G$1" pin="7"/>
-<pinref part="SUPPLY12" gate="1" pin="VCC"/>
-<wire x1="22.86" y1="40.64" x2="22.86" y2="38.1" width="0.1524" layer="91"/>
 </segment>
 <segment>
@@
 <pinref part="JP5" gate="A" pin="6"/>
 <wire x1="-93.98" y1="243.84" x2="-88.9" y2="243.84" width="0.1524" layer="91"/>
-<label x="-88.9" y="243.84" size="1.778" layer="95"/>
+<label x="-86.36" y="243.84" size="1.778" layer="95"/>
+</segment>
+<segment>
+<wire x1="80.01" y1="99.06" x2="91.44" y2="99.06" width="0.1524" layer="91"/>
+<label x="82.55" y="99.06" size="1.778" layer="95"/>
+<pinref part="ATMEGA328" gate="G$1" pin="PB2(SS/OC1B)"/>
 </segment>
 </net>
@@
 </segment>
 </net>
+<net name="3V3R" class="0">
+<segment>
+<pinref part="J1" gate="G$1" pin="3"/>
+<wire x1="289.56" y1="91.44" x2="309.88" y2="91.44" width="0.1524" layer="91"/>
+<label x="287.02" y="91.44" size="1.778" layer="95"/>
+</segment>
+<segment>
+<wire x1="193.04" y1="71.12" x2="200.66" y2="71.12" width="0.1524" layer="91"/>
+<wire x1="200.66" y1="71.12" x2="215.9" y2="71.12" width="0.1524" layer="91"/>
+<pinref part="IC3" gate="G$1" pin="VO"/>
+<wire x1="193.04" y1="71.12" x2="193.04" y2="76.2" width="0.2032" layer="91"/>
+<pinref part="C4" gate="G$1" pin="1"/>
+<junction x="193.04" y="71.12"/>
+<pinref part="C3" gate="G$1" pin="1"/>
+<junction x="200.66" y="71.12"/>
+<label x="193.04" y="78.74" size="1.778" layer="95"/>
+</segment>
+<segment>
+<pinref part="J2" gate="G$1" pin="7"/>
+<wire x1="22.86" y1="40.64" x2="22.86" y2="38.1" width="0.1524" layer="91"/>
+<label x="20.32" y="40.64" size="1.778" layer="95"/>
+</segment>
+</net>

Commit message: update
Parts:
- renumbered BATTPOWER to M1, REMOTE to M3, RTC-DS3231 to RTC, SDPWER to M2, U$1 to SD, U$2 to D1
Connections:
- removed net D11_MOSI: ATMEGA328.PB3(MOSI/OC2), ISP.4
- removed net D12_MISO: ATMEGA328.PB4(MISO), ISP.1
- removed net D13_SCK: ATMEGA328.PB5(SCK), ISP.3
- removed net D5/RTC: RTC.INT/SQW
- removed net VBAT: JP5.14
- net A2: now also JP5.10; no longer JP5.8
- net A3: now also JP5.8
- net AREF: now also JP5.2; no longer JP5.4
- net D10: now also JP5.4; no longer JP5.6
- net D3: now also JP5.6; no longer JP5.10
- net D5: now also RTC.INT/SQW
- net MISO: now also ATMEGA328.PB4(MISO), ISP.1
- net MOSI: now also ATMEGA328.PB3(MOSI/OC2), ISP.4
- net N$7: no longer JP5.2
- net PWR: now also JP5.14
- net SCK: now also ATMEGA328.PB5(SCK), ISP.3

Commit message: update
Parts:
- renumbered SD to MICROSD
Changed lines of the file:
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@@
 <part name="P+6" library="supply1" deviceset="VCC" device=""/>
 <part name="GND4" library="supply1" deviceset="GND" device=""/>
-<part name="SD" library="hrs_DM3D-SF" deviceset="MICROSD-HRS_DM3D" device=""/>
+<part name="MICROSD" library="hrs_DM3D-SF" deviceset="MICROSD-HRS_DM3D" device=""/>
 <part name="M1" library="zetex" deviceset="PMOSSOT23" device="" value="FDN340P"/>
 <part name="GND7" library="SparkFun" deviceset="GND" device=""/>
@@
 <instance part="P+6" gate="VCC" x="-109.982" y="267.97"/>
 <instance part="GND4" gate="1" x="413.512" y="213.868"/>
-<instance part="SD" gate="G$1" x="290.322" y="229.362"/>
+<instance part="MICROSD" gate="G$1" x="290.322" y="229.362"/>
 <instance part="M1" gate="A" x="420.116" y="257.048" rot="MR270"/>
 <instance part="GND7" gate="1" x="398.018" y="257.048" rot="R270"/>
@@
 </segment>
 <segment>
-<pinref part="SD" gate="G$1" pin="GND"/>
+<pinref part="MICROSD" gate="G$1" pin="GND"/>
 <pinref part="GND9" gate="1" pin="GND"/>
 <wire x1="309.372" y1="242.062" x2="308.102" y2="242.062" width="0.1524" layer="91"/>
 </segment>
 <segment>
-<pinref part="SD" gate="G$1" pin="SW_B"/>
+<pinref part="MICROSD" gate="G$1" pin="SW_B"/>
 <pinref part="GND10" gate="1" pin="GND"/>
 <wire x1="308.102" y1="209.55" x2="308.102" y2="214.122" width="0.1524" layer="91"/>
-<pinref part="SD" gate="G$1" pin="GND2"/>
-<pinref part="SD" gate="G$1" pin="GND3"/>
+<pinref part="MICROSD" gate="G$1" pin="GND2"/>
+<pinref part="MICROSD" gate="G$1" pin="GND3"/>
 <wire x1="308.102" y1="226.822" x2="308.102" y2="224.282" width="0.1524" layer="91"/>
-<pinref part="SD" gate="G$1" pin="GND4"/>
+<pinref part="MICROSD" gate="G$1" pin="GND4"/>
 <wire x1="308.102" y1="224.282" x2="308.102" y2="221.742" width="0.1524" layer="91"/>
-<pinref part="SD" gate="G$1" pin="SW_A"/>
+<pinref part="MICROSD" gate="G$1" pin="SW_A"/>
 <wire x1="308.102" y1="221.742" x2="308.102" y2="216.662" width="0.1524" layer="91"/>
 <wire x1="308.102" y1="216.662" x2="308.102" y2="214.122" width="0.1524" layer="91"/>
@@
 <junction x="308.102" y="216.662"/>
 <junction x="308.102" y="214.122"/>
-<pinref part="SD" gate="G$1" pin="GND1"/>
+<pinref part="MICROSD" gate="G$1" pin="GND1"/>
 <wire x1="308.102" y1="229.362" x2="308.102" y2="226.822" width="0.1524" layer="91"/>
 <junction x="308.102" y="226.822"/>
@@
 </segment>
 <segment>
-<pinref part="SD" gate="G$1" pin="CD/DAT3"/>
+<pinref part="MICROSD" gate="G$1" pin="CD/DAT3"/>
 <wire x1="308.102" y1="236.982" x2="318.77" y2="236.982" width="0.1524" layer="91"/>
 <label x="320.802" y="236.982" size="1.778" layer="95"/>
@@
 <net name="SCK" class="0">
 <segment>
-<pinref part="SD" gate="G$1" pin="CLK"/>
+<pinref part="MICROSD" gate="G$1" pin="CLK"/>
 <wire x1="308.102" y1="247.142" x2="319.024" y2="247.142" width="0.1524" layer="91"/>
 <label x="320.802" y="247.142" size="1.778" layer="95"/>
@@
 <net name="MISO" class="0">
 <segment>
-<pinref part="SD" gate="G$1" pin="DAT0"/>
+<pinref part="MICROSD" gate="G$1" pin="DAT0"/>
 <wire x1="308.102" y1="249.682" x2="319.024" y2="249.682" width="0.1524" layer="91"/>
 <label x="320.802" y="249.682" size="1.778" layer="95"/>
@@
 <net name="MOSI" class="0">
 <segment>
-<pinref part="SD" gate="G$1" pin="CMD"/>
+<pinref part="MICROSD" gate="G$1" pin="CMD"/>
 <wire x1="308.102" y1="239.522" x2="318.77" y2="239.522" width="0.1524" layer="91"/>
 <label x="320.802" y="239.522" size="1.778" layer="95"/>
@@
 <net name="N$16" class="0">
 <segment>
-<pinref part="SD" gate="G$1" pin="DAT1"/>
+<pinref part="MICROSD" gate="G$1" pin="DAT1"/>
 <wire x1="308.102" y1="252.222" x2="308.102" y2="254.762" width="0.1524" layer="91"/>
 <wire x1="308.102" y1="254.762" x2="343.408" y2="254.762" width="0.1524" layer="91"/>
@@
 <net name="N$18" class="0">
 <segment>
-<pinref part="SD" gate="G$1" pin="DAT2"/>
+<pinref part="MICROSD" gate="G$1" pin="DAT2"/>
 <wire x1="308.102" y1="234.442" x2="343.408" y2="234.442" width="0.1524" layer="91"/>
 <pinref part="R8" gate="G$1" pin="1"/>
@@
 <junction x="354.076" y="271.272"/>
 <wire x1="354.076" y1="271.272" x2="354.076" y2="244.602" width="0.1524" layer="91"/>
-<pinref part="SD" gate="G$1" pin="VDD"/>
+<pinref part="MICROSD" gate="G$1" pin="VDD"/>
 <wire x1="308.102" y1="244.602" x2="343.408" y2="244.602" width="0.1524" layer="91"/>
 <pinref part="R7" gate="G$1" pin="1"/>
